File: Kicad/Frame_PCB/V0-UmbilicalBoard.kicad_pcb (KiCad board)
At the start: 2 copper layers, 122 x 37 mm, 17 parts, among them J1 Conn_02x10_Top_Bottom, J10 Neopixel Strip 1, J11 Neopixel Strip 1, J12 Neopixel Out, J13 Accelerometer, J2 Motor, J3 Hotend Fan, J4 Part Cooling Fan, J5 Heater, J6 Thermistor, J7 X-Endstop, J8 Chamber Thermistor, J9 Neopixel (from controller)

Commit message: Added missing 3D model for Molex MicroFit
Parts:
- J1: footprint Connector_Molex:Molex_Micro-Fit_3.0_43045-2012_2x10_P3.00mm_Vertical -> V0-UmbilicalBoard:Molex_Micro-Fit_3.0_43045-2012_2x10_P3.00mm_Vertical
Changed lines of the file:
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@@
   (net 25 "Net-(J1-Pad19)")
   (net 26 "Net-(J1-Pad20)")
-  (footprint "Connector_Molex:Molex_Micro-Fit_3.0_43045-2012_2x10_P3.00mm_Vertical" (layer "F.Cu")
+  (footprint "V0-UmbilicalBoard:Molex_Micro-Fit_3.0_43045-2012_2x10_P3.00mm_Vertical" (layer "F.Cu")
     (at 113.5 101.5 180)
     (descr "Molex Micro-Fit 3.0 Connector System, 43045-2012 (compatible alternatives: 43045-2013, 43045-2024), 10 Pins per row (http://www.molex.com/pdm_docs/sd/430450212_sd.pdf), generated with kicad-footprint-generator")
@@
       (effects (font (size 1 1) (thickness 0.15)))
     )
+    (fp_line (start -2.015 -2.58) (end -2.015 -2.08) (layer "F.SilkS") (width 0.12))
+    (fp_line (start 29.015 -2.58) (end 30.435 -2.58) (layer "F.SilkS") (width 0.12))
+    (fp_line (start -3.435 -2.58) (end -2.015 -2.58) (layer "F.SilkS") (width 0.12))
+    (fp_line (start -2.015 -2.08) (end 29.015 -2.08) (layer "F.SilkS") (width 0.12))
+    (fp_line (start 30.435 -2.58) (end 30.435 3.18) (layer "F.SilkS") (width 0.12))
+    (fp_line (start -3.435 5.01) (end 30.435 5.01) (layer "F.SilkS") (width 0.12))
+    (fp_line (start -3.435 3.18) (end -3.435 -2.58) (layer "F.SilkS") (width 0.12))
+    (fp_line (start -3.435 4.7) (end -3.435 5.01) (layer "F.SilkS") (width 0.12))
     (fp_line (start 30.435 5.01) (end 30.435 4.7) (layer "F.SilkS") (width 0.12))
     (fp_line (start 29.015 -2.08) (end 29.015 -2.58) (layer "F.SilkS") (width 0.12))
-    (fp_line (start -3.435 4.7) (end -3.435 5.01) (layer "F.SilkS") (width 0.12))
-    (fp_line (start -3.435 3.18) (end -3.435 -2.58) (layer "F.SilkS") (width 0.12))
-    (fp_line (start 30.435 -2.58) (end 30.435 3.18) (layer "F.SilkS") (width 0.12))
-    (fp_line (start -3.435 5.01) (end 30.435 5.01) (layer "F.SilkS") (width 0.12))
-    (fp_line (start -2.015 -2.58) (end -2.015 -2.08) (layer "F.SilkS") (width 0.12))
-    (fp_line (start -2.015 -2.08) (end 29.015 -2.08) (layer "F.SilkS") (width 0.12))
-    (fp_line (start -3.435 -2.58) (end -2.015 -2.58) (layer "F.SilkS") (width 0.12))
-    (fp_line (start 29.015 -2.58) (end 30.435 -2.58) (layer "F.SilkS") (width 0.12))
+    (fp_line (start -3.82 6.8) (end -3.82 -2.97) (layer "F.CrtYd") (width 0.05))
     (fp_line (start -3.82 -2.97) (end 30.82 -2.97) (layer "F.CrtYd") (width 0.05))
-    (fp_line (start -3.82 6.8) (end -3.82 -2.97) (layer "F.CrtYd") (width 0.05))
     (fp_line (start 30.82 -2.97) (end 30.82 6.8) (layer "F.CrtYd") (width 0.05))
     (fp_line (start 30.82 6.8) (end -3.82 6.8) (layer "F.CrtYd") (width 0.05))
-    (fp_line (start 14.2 6.3) (end 14.2 4.9) (layer "F.Fab") (width 0.1))
+    (fp_line (start 12.8 4.9) (end 12.8 6.3) (layer "F.Fab") (width 0.1))
     (fp_line (start 29.125 -1.97) (end -2.125 -1.97) (layer "F.Fab") (width 0.1))
-    (fp_line (start -2.125 -1.97) (end -2.125 -2.47) (layer "F.Fab") (width 0.1))
+    (fp_line (start -3.325 -1.34) (end -2.125 -1.97) (layer "F.Fab") (width 0.1))
     (fp_line (start 30.325 -2.47) (end 29.125 -2.47) (layer "F.Fab") (width 0.1))
     (fp_line (start 29.125 -2.47) (end 29.125 -1.97) (layer "F.Fab") (width 0.1))
-    (fp_line (start -2.125 -2.47) (end -3.325 -2.47) (layer "F.Fab") (width 0.1))
-    (fp_line (start 30.325 -1.34) (end 29.125 -1.97) (layer "F.Fab") (width 0.1))
-    (fp_line (start 12.8 4.9) (end 12.8 6.3) (layer "F.Fab") (width 0.1))
+    (fp_line (start 0 -1.262893) (end 0.5 -1.97) (layer "F.Fab") (width 0.1))
+    (fp_line (start 30.325 4.9) (end 30.325 -2.47) (layer "F.Fab") (width 0.1))
     (fp_line (start -0.5 -1.97) (end 0 -1.262893) (layer "F.Fab") (width 0.1))
+    (fp_line (start 14.2 6.3) (end 14.2 4.9) (layer "F.Fab") (width 0.1))
     (fp_line (start -3.325 -2.47) (end -3.325 4.9) (layer "F.Fab") (width 0.1))
     (fp_line (start -3.325 4.9) (end 30.325 4.9) (layer "F.Fab") (width 0.1))
-    (fp_line (start 0 -1.262893) (end 0.5 -1.97) (layer "F.Fab") (width 0.1))
+    (fp_line (start 30.325 -1.34) (end 29.125 -1.97) (layer "F.Fab") (width 0.1))
+    (fp_line (start -2.125 -1.97) (end -2.125 -2.47) (layer "F.Fab") (width 0.1))
+    (fp_line (start -2.125 -2.47) (end -3.325 -2.47) (layer "F.Fab") (width 0.1))
     (fp_line (start 12.8 6.3) (end 14.2 6.3) (layer "F.Fab") (width 0.1))
-    (fp_line (start 30.325 4.9) (end 30.325 -2.47) (layer "F.Fab") (width 0.1))
-    (fp_line (start -3.325 -1.34) (end -2.125 -1.97) (layer "F.Fab") (width 0.1))
+    (pad "" np_thru_hole circle (at 30 3.94 180) (size 1 1) (drill 1) (layers *.Cu *.Mask))
     (pad "" np_thru_hole circle (at -3 3.94 180) (size 1 1) (drill 1) (layers *.Cu *.Mask))
-    (pad "" np_thru_hole circle (at 30 3.94 180) (size 1 1) (drill 1) (layers *.Cu *.Mask))
-    (pad "1" thru_hole roundrect (at 0 0 180) (size 1.5 1.5) (drill 1) (layers *.Cu *.Mask) (roundrect_rratio 0.1666673333)
+    (pad "1" thru_hole roundrect (at 0 0 180) (size 1.5 1.5) (drill 1) (layers *.Cu *.Mask) (roundrect_rratio 0.166667)
       (net 17 "/ADXL_GND") (pinfunction "Pin_1") (pintype "passive"))
     (pad "2" thru_hole circle (at 3 0 180) (size 1.5 1.5) (drill 1) (layers *.Cu *.Mask)
@@
     (pad "20" thru_hole circle (at 27 3 180) (size 1.5 1.5) (drill 1) (layers *.Cu *.Mask)
       (net 26 "Net-(J1-Pad20)") (pinfunction "Pin_20") (pintype "passive"))
-    (model "${KISYS3DMOD}/Connector_Molex.3dshapes/Molex_Micro-Fit_3.0_43045-2012_2x10_P3.00mm_Vertical.wrl"
-      (offset (xyz 0 0 0))
+    (model "${KIPRJMOD}/Library/3D_Packages/430452012.stp"
+      (offset (xyz 13.5 -1.5 5))
       (scale (xyz 1 1 1))
-      (rotate (xyz 0 0 0))
+      (rotate (xyz 0 0 180))
     )
   )
