File: Kicad/Frame_PCB/V0-UmbilicalBoard.kicad_sch (KiCad schematic)
At the start: 17 parts, among them J1 Conn_02x10_Top_Bottom, J10 Neopixel Strip 1, J11 Neopixel Strip 1, J12 Neopixel Out, J13 Accelerometer, J2 Motor, J3 Hotend Fan, J4 Part Cooling Fan, J5 Heater, J6 Thermistor, J7 X-Endstop, J8 Chamber Thermistor, J9 Neopixel (from controller)

Commit message: Added missing 3D model for Molex MicroFit
Parts:
- J1: footprint Connector_Molex:Molex_Micro-Fit_3.0_43045-2012_2x10_P3.00mm_Vertical -> V0-UmbilicalBoard:Molex_Micro-Fit_3.0_43045-2012_2x10_P3.00mm_Vertical
Changed lines of the file:
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@@
     (property "Reference" "J1" (id 0) (at 116.84 52.07 0))
     (property "Value" "Conn_02x10_Top_Bottom" (id 1) (at 116.84 54.61 0))
-    (property "Footprint" "Connector_Molex:Molex_Micro-Fit_3.0_43045-2012_2x10_P3.00mm_Vertical" (id 2) (at 115.57 68.58 0)
+    (property "Footprint" "V0-UmbilicalBoard:Molex_Micro-Fit_3.0_43045-2012_2x10_P3.00mm_Vertical" (id 2) (at 115.57 68.58 0)
       (effects (font (size 1.27 1.27)) hide)
     )
@@
     )
     (path "/b57ff189-3eae-4dfe-9050-48699ec7dcd8"
-      (reference "J1") (unit 1) (value "Conn_02x10_Top_Bottom") (footprint "Connector_Molex:Molex_Micro-Fit_3.0_43045-2012_2x10_P3.00mm_Vertical")
+      (reference "J1") (unit 1) (value "Conn_02x10_Top_Bottom") (footprint "V0-UmbilicalBoard:Molex_Micro-Fit_3.0_43045-2012_2x10_P3.00mm_Vertical")
     )
     (path "/00000000-0000-0000-0000-0000607f8393"
